Commit message: daily checkin
daily checkin - tea time

File: urdf/azure_kinect.urdf.xacro (robot description, xacro)
@@ -14,9 +14,57 @@
   <material name="grey">
     <color rgba="0.6 0.6 0.6 1" />
+ </material>
+  <material name="gray">
+    <color rgba="0.2 0.2 0.2 1" />
+  </material>
+  <material name="brightRed">
+    <color rgba="1.0 0 0 1.0" />
   </material>
   <material name="white">
     <color rgba="0.9 0.9 0.9 1" />
   </material>
-  <link name="$(arg tf_prefix)camera_body">
+    <material name="orange">
+    <color rgba="1.0 0.5 0.2 1" />
+  </material>
+  <link name="camera_base">
+    <visual>
+      <origin xyz="-0.013 0. 0." />
+      <geometry>
+        <box size="0.026 0.103 0.039" />
+      </geometry>
+	  <parent link="map" />
+      <material name="brightRed" />
+    </visual>
+  </link>
+  <link name="depth_camera_link">
+    <visual>
+      <origin xyz="0 0 0" />
+      <geometry>
+        <cylinder length="0.05" radius="0.03" />
+      </geometry>
+      <material name="gray" />
+    </visual>
+  </link>
+  <link name="imu_link">
+    <visual>
+      <origin xyz="0 0 0" />
+      <geometry>
+        <box size="0.06 0.04 0.02" />
+      </geometry>
+      <material name="orange" />
+    </visual>
+  </link>
+  <joint name="imu_link_joint" type="fixed">
+    <parent link="camera_base" />
+    <child link="imu_link" />
+    <origin xyz="0 0 0" />
+  </joint>
+    <joint name="depth_camera_link_joint" type="fixed">
+    <parent link="camera_base" />
+    <child link="depth_camera_link" />
+	<!--origin rpy="0 -1.570796 3.141593" xyz="0.000 0 0.0000"  -->
+    <origin rpy="0 1.570796 0" xyz="0.000 0 0.0000" />
+  </joint>
+  <link name="camera_body">
     <visual>
       <origin xyz="0. 0. 0." />
@@ -27,14 +75,5 @@
     </visual>
   </link>
-  <link name="$(arg tf_prefix)camera_base">
-    <visual>
-      <origin xyz="-0.013 0. 0." />
-      <geometry>
-        <box size="0.026 0.103 0.039" />
-      </geometry>
-      <material name="grey" />
-    </visual>
-  </link>
-  <link name="$(arg tf_prefix)camera_visor">
+  <link name="camera_visor">
     <visual>
       <origin xyz="-0.0128 0. 0." />
@@ -45,12 +84,12 @@
     </visual>
   </link>
-  <joint name="$(arg tf_prefix)camera_base_to_body" type="fixed">
-    <parent link="$(arg tf_prefix)camera_base" />
-    <child link="$(arg tf_prefix)camera_body" />
+  <joint name="camera_base_to_body" type="fixed">
+    <parent link="camera_base" />
+    <child link="camera_body" />
     <origin xyz="-0.0757 0. 0.008" rpy="0. 0. 0." />
   </joint>
   <joint name="$(arg tf_prefix)camera_base_to_visor" type="fixed">
-    <parent link="$(arg tf_prefix)camera_base" />
-    <child link="$(arg tf_prefix)camera_visor" />
+    <parent link="camera_base" />
+    <child link="camera_visor" />
     <origin xyz="0. 0. 0." rpy="0. 0. 0." />
   </joint>

Commit message: daily checkin
daily checkin

File: urdf/azure_kinect.urdf.xacro (robot description, xacro)
@@ -33,5 +33,5 @@
         <box size="0.026 0.103 0.039" />
       </geometry>
-	  <parent link="map" />
+	  <parent link="odom" />
       <material name="brightRed" />
     </visual>
@@ -64,5 +64,5 @@
     <child link="depth_camera_link" />
 	<!--origin rpy="0 -1.570796 3.141593" xyz="0.000 0 0.0000"  -->
-    <origin rpy="0 1.570796 0" xyz="0.000 0 0.0000" />
+    <origin rpy="0 0 0" xyz="0.000 0 0.0000" />
   </joint>
   <link name="camera_body">

Commit message: daily checkin
fix up k4a geometry /sensor pipeline

File: urdf/azure_kinect.urdf.xacro (robot description, xacro)
@@ -27,5 +27,5 @@
     <color rgba="1.0 0.5 0.2 1" />
   </material>
-  <link name="camera_base">
+  <link name="base_link">
     <visual>
       <origin xyz="-0.013 0. 0." />
@@ -47,4 +47,5 @@
   </link>
   <link name="imu_link">
+      <parent link="base_link" />
     <visual>
       <origin xyz="0 0 0" />
@@ -55,14 +56,14 @@
     </visual>
   </link>
-  <joint name="imu_link_joint" type="fixed">
-    <parent link="camera_base" />
+  <joint name="base_imu_joint" type="fixed">
+    <parent link="base_link" />
     <child link="imu_link" />
     <origin xyz="0 0 0" />
   </joint>
-    <joint name="depth_camera_link_joint" type="fixed">
-    <parent link="camera_base" />
+  <joint name="base_depth_joint" type="fixed">
+    <parent link="base_link" />
     <child link="depth_camera_link" />
 	<!--origin rpy="0 -1.570796 3.141593" xyz="0.000 0 0.0000"  -->
-    <origin rpy="0 0 0" xyz="0.000 0 0.0000" />
+    <origin rpy="0 -1.570796 0" xyz="0.000 0 0.0000" />
   </joint>
   <link name="camera_body">
@@ -84,11 +85,11 @@
     </visual>
   </link>
-  <joint name="camera_base_to_body" type="fixed">
-    <parent link="camera_base" />
+  <joint name="base_to_body" type="fixed">
+    <parent link="base_link" />
     <child link="camera_body" />
     <origin xyz="-0.0757 0. 0.008" rpy="0. 0. 0." />
   </joint>
-  <joint name="$(arg tf_prefix)camera_base_to_visor" type="fixed">
-    <parent link="camera_base" />
+  <joint name="base_to_visor" type="fixed">
+    <parent link="base_link" />
     <child link="camera_visor" />
     <origin xyz="0. 0. 0." rpy="0. 0. 0." />

Commit message: daily checkin
daily checkin

File: urdf/azure_kinect.urdf.xacro (robot description, xacro)
@@ -28,4 +28,5 @@
   </material>
   <link name="base_link">
+  	  <parent link="odom" />
     <visual>
       <origin xyz="-0.013 0. 0." />
@@ -33,9 +34,19 @@
         <box size="0.026 0.103 0.039" />
       </geometry>
-	  <parent link="odom" />
       <material name="brightRed" />
     </visual>
   </link>
+    <link name="imu_link">
+      <parent link="odom" />
+    <visual>
+      <origin xyz="0 0 0" />
+      <geometry>
+        <box size="0.06 0.04 0.02" />
+      </geometry>
+      <material name="orange" />
+    </visual>
+  </link>
   <link name="depth_camera_link">
+    <parent link="odom" />
     <visual>
       <origin xyz="0 0 0" />
@@ -46,25 +57,4 @@
     </visual>
   </link>
-  <link name="imu_link">
-      <parent link="base_link" />
-    <visual>
-      <origin xyz="0 0 0" />
-      <geometry>
-        <box size="0.06 0.04 0.02" />
-      </geometry>
-      <material name="orange" />
-    </visual>
-  </link>
-  <joint name="base_imu_joint" type="fixed">
-    <parent link="base_link" />
-    <child link="imu_link" />
-    <origin xyz="0 0 0" />
-  </joint>
-  <joint name="base_depth_joint" type="fixed">
-    <parent link="base_link" />
-    <child link="depth_camera_link" />
-	<!--origin rpy="0 -1.570796 3.141593" xyz="0.000 0 0.0000"  -->
-    <origin rpy="0 -1.570796 0" xyz="0.000 0 0.0000" />
-  </joint>
   <link name="camera_body">
     <visual>
@@ -95,3 +85,14 @@
     <origin xyz="0. 0. 0." rpy="0. 0. 0." />
   </joint>
+  <joint name="base_imu_joint" type="fixed">
+    <parent link="base_link" />
+    <child link="imu_link" />
+    <origin xyz="0 0 0" />
+  </joint>
+  <joint name="base_depth_joint" type="fixed">
+    <parent link="base_link" />
+    <child link="depth_camera_link" />
+	<!--origin rpy="0 -1.570796 3.141593" xyz="0.000 0 0.0000"  -->
+    <origin rpy="0 -1.570796 0" xyz="0.000 0 0.0000" />
+  </joint>
 </robot>

Commit message: fix for cartographer integration
fix for cartographer

File: urdf/azure_kinect.urdf.xacro (robot description, xacro)
@@ -48,5 +48,5 @@
   </link>
   <link name="depth_camera_link">
-    <parent link="odom" />
+    <parent link="map" />
     <visual>
       <origin xyz="0 0 0" />

Commit message: fix up topic names from driver
fix up topic names from driver

File: urdf/azure_kinect.urdf.xacro (robot description, xacro)
@@ -37,5 +37,5 @@
     </visual>
   </link>
-    <link name="imu_link">
+    <link name="imu">
       <parent link="odom" />
     <visual>
@@ -86,7 +86,7 @@
   </joint>
   <joint name="base_imu_joint" type="fixed">
-    <parent link="base_link" />
-    <child link="imu_link" />
-    <origin xyz="0 0 0" />
+    <parent link="depth_camera_link" />
+    <child link="imu" />
+    <origin rpy="0 0 0" xyz="0 0 0" />
   </joint>
   <joint name="base_depth_joint" type="fixed">
@@ -94,5 +94,5 @@
     <child link="depth_camera_link" />
 	<!--origin rpy="0 -1.570796 3.141593" xyz="0.000 0 0.0000"  -->
-    <origin rpy="0 -1.570796 0" xyz="0.000 0 0.0000" />
+    <origin rpy="0 0 0" xyz="0.000 0 0.0000" />
   </joint>
 </robot>

Commit message: daily checkin
daily checkin

File: urdf/azure_kinect.urdf.xacro (robot description, xacro)
@@ -38,5 +38,5 @@
   </link>
     <link name="imu">
-      <parent link="odom" />
+      <parent link="base_link" />
     <visual>
       <origin xyz="0 0 0" />
@@ -47,5 +47,5 @@
     </visual>
   </link>
-  <link name="depth_camera_link">
+  <link name="odom">
     <parent link="map" />
     <visual>
@@ -86,11 +86,11 @@
   </joint>
   <joint name="base_imu_joint" type="fixed">
-    <parent link="depth_camera_link" />
+    <parent link="base_link" />
     <child link="imu" />
     <origin rpy="0 0 0" xyz="0 0 0" />
   </joint>
-  <joint name="base_depth_joint" type="fixed">
+  <joint name="base_odom_joint" type="fixed">
     <parent link="base_link" />
-    <child link="depth_camera_link" />
+    <child link="odom" />
 	<!--origin rpy="0 -1.570796 3.141593" xyz="0.000 0 0.0000" -->
     <origin rpy="0 0 0" xyz="0.000 0 0.0000" />

Commit message: daily checkin
daily checkin

File: urdf/azure_kinect.urdf.xacro (robot description, xacro)
@@ -37,6 +37,5 @@
     </visual>
   </link>
-    <link name="imu">
-      <parent link="base_link" />
+  <link name="imu">
     <visual>
       <origin xyz="0 0 0" />
@@ -45,14 +44,4 @@
       </geometry>
       <material name="orange" />
-    </visual>
-  </link>
-  <link name="odom">
-    <parent link="map" />
-    <visual>
-      <origin xyz="0 0 0" />
-      <geometry>
-        <cylinder length="0.05" radius="0.03" />
-      </geometry>
-      <material name="gray" />
     </visual>
   </link>
@@ -66,22 +55,8 @@
     </visual>
   </link>
-  <link name="camera_visor">
-    <visual>
-      <origin xyz="-0.0128 0. 0." />
-      <geometry>
-        <box size="0.026 0.101 0.037" />
-      </geometry>
-      <material name="black" />
-    </visual>
-  </link>
   <joint name="base_to_body" type="fixed">
     <parent link="base_link" />
     <child link="camera_body" />
     <origin xyz="-0.0757 0. 0.008" rpy="0. 0. 0." />
-  </joint>
-  <joint name="base_to_visor" type="fixed">
-    <parent link="base_link" />
-    <child link="camera_visor" />
-    <origin xyz="0. 0. 0." rpy="0. 0. 0." />
   </joint>
   <joint name="base_imu_joint" type="fixed">
@@ -90,9 +65,3 @@
     <origin rpy="0 0 0" xyz="0 0 0" />
   </joint>
-  <joint name="base_odom_joint" type="fixed">
-    <parent link="base_link" />
-    <child link="odom" />
-	<!--origin rpy="0 -1.570796 3.141593" xyz="0.000 0 0.0000" -->
-    <origin rpy="0 0 0" xyz="0.000 0 0.0000" />
-  </joint>
 </robot>

Commit message: checkin before build
checkin before build

File: urdf/azure_kinect.urdf.xacro (robot description, xacro)
@@ -37,5 +37,5 @@
     </visual>
   </link>
-  <link name="imu">
+  <link name="imu_link">
     <visual>
       <origin xyz="0 0 0" />
@@ -62,5 +62,5 @@
   <joint name="base_imu_joint" type="fixed">
     <parent link="base_link" />
-    <child link="imu" />
+    <child link="imu_link" />
     <origin rpy="0 0 0" xyz="0 0 0" />
   </joint>

Commit message: checkin prior to build
checkin prior to build

File: urdf/azure_kinect.urdf.xacro (robot description, xacro)
@@ -46,4 +46,13 @@
     </visual>
   </link>
+  <link name="depth_camera_link">
+    <visual>
+      <origin xyz="0 0 0" />
+      <geometry>
+        <cylinder length="0.05" radius="0.03" />
+      </geometry>
+      <material name="gray" />
+    </visual>
+  </link>
   <link name="camera_body">
     <visual>
@@ -55,4 +64,14 @@
     </visual>
   </link>
+   <joint name="depth_camera_link_joint" type="fixed">
+    <parent link="base_link" />
+    <child link="depth_camera_link" />
+    <origin xyz="0.0 0 0.0" />
+  </joint>
+  <joint name="imu_link_joint" type="fixed">
+    <parent link="base_link" />
+    <child link="imu_link" />
+    <origin rpy="0 0 0" xyz="0 0 0" />
+  </joint>
   <joint name="base_to_body" type="fixed">
     <parent link="base_link" />
@@ -60,8 +79,3 @@
     <origin xyz="-0.0757 0. 0.008" rpy="0. 0. 0." />
   </joint>
-  <joint name="base_imu_joint" type="fixed">
-    <parent link="base_link" />
-    <child link="imu_link" />
-    <origin rpy="0 0 0" xyz="0 0 0" />
-  </joint>
 </robot>

Commit message: robot config like demo
robot config like demo

File: urdf/azure_kinect.urdf.xacro (robot description, xacro)
@@ -27,14 +27,4 @@
     <color rgba="1.0 0.5 0.2 1" />
   </material>
-  <link name="base_link">
-  	  <parent link="odom" />
-    <visual>
-      <origin xyz="-0.013 0. 0." />
-      <geometry>
-        <box size="0.026 0.103 0.039" />
-      </geometry>
-      <material name="brightRed" />
-    </visual>
-  </link>
   <link name="imu_link">
     <visual>
@@ -46,5 +36,5 @@
     </visual>
   </link>
-  <link name="depth_camera_link">
+  <link name="horizontal_laser_link">
     <visual>
       <origin xyz="0 0 0" />
@@ -64,13 +54,14 @@
     </visual>
   </link>
-   <joint name="depth_camera_link_joint" type="fixed">
-    <parent link="base_link" />
-    <child link="depth_camera_link" />
-    <origin xyz="0.0 0 0.0" />
-  </joint>
+  <link name="base_link" />
   <joint name="imu_link_joint" type="fixed">
     <parent link="base_link" />
     <child link="imu_link" />
     <origin rpy="0 0 0" xyz="0 0 0" />
+  </joint>
+  <joint name="horizontal_laser_link_joint" type="fixed">
+    <parent link="base_link" />
+    <child link="horizontal_laser_link" />
+    <origin xyz="0.0 0 0.0" />
   </joint>
   <joint name="base_to_body" type="fixed">

Commit message: update initial pose
update initial pose

File: urdf/azure_kinect.urdf.xacro (robot description, xacro)
@@ -58,15 +58,15 @@
     <parent link="base_link" />
     <child link="imu_link" />
-    <origin rpy="0 0 0" xyz="0 0 0" />
+    <origin rpy="0 1.57 -3.1415" xyz="0 0 0" />
   </joint>
   <joint name="horizontal_laser_link_joint" type="fixed">
     <parent link="base_link" />
     <child link="horizontal_laser_link" />
-    <origin xyz="0.0 0 0.0" />
+    <origin rpy="0 0 0.0" xyz="0.0 0.0 0.0" />
   </joint>
   <joint name="base_to_body" type="fixed">
     <parent link="base_link" />
     <child link="camera_body" />
-    <origin xyz="-0.0757 0. 0.008" rpy="0. 0. 0." />
+    <origin xyz="0.0 0. 0.0" rpy="0. 0. 0." />
   </joint>
 </robot>

Commit message: forward -x for azure
forward -x for azure

File: urdf/azure_kinect.urdf.xacro (robot description, xacro)
@@ -58,5 +58,5 @@
     <parent link="base_link" />
     <child link="imu_link" />
-    <origin rpy="0 1.57 -3.1415" xyz="0 0 0" />
+    <origin rpy="-3.1415 0 0" xyz="0 0 0" />
   </joint>
   <joint name="horizontal_laser_link_joint" type="fixed">

Commit message: daily checkin
daily checkin

File: urdf/azure_kinect.urdf.xacro (robot description, xacro)
@@ -58,5 +58,5 @@
     <parent link="base_link" />
     <child link="imu_link" />
-    <origin rpy="-3.1415 0 0" xyz="0 0 0" />
+    <origin rpy="3.1415 0 0" xyz="0 0 0" />
   </joint>
   <joint name="horizontal_laser_link_joint" type="fixed">
